Commit message: camera gazebo plugin added ,  rviz and gazebo meshes loading bug fixed

File: src/robot_description/urdf/bumperbot.urdf.xacro (robot description, xacro)
@@ -21,5 +21,5 @@
             <geometry>
                 <!-- <mesh filename="package://robot_description/meshes/base_link.STL" scale="1 1 1"/> -->
-                <mesh filename="$(find robot_description)/meshes/base_link.STL"/>
+                <mesh filename="file://$(find robot_description)/meshes/base_link.STL"/>
             </geometry>
         </visual>
@@ -28,5 +28,5 @@
             <geometry>
                 <!-- <mesh filename="package://robot_description/meshes/base_link.STL" scale="1 1 1"/> -->
-                <mesh filename="$(find robot_description)/meshes/base_link.STL"/>
+                <mesh filename="file://$(find robot_description)/meshes/base_link.STL"/>
             </geometry>
         </collision>
@@ -50,5 +50,5 @@
             <geometry>
                 <!-- <mesh filename="package://robot_description/meshes/wheel_right_link.STL" scale="1 1 1"/> -->
-                <mesh filename="$(find robot_description)/meshes/wheel_right_link.STL"/>
+                <mesh filename="file://$(find robot_description)/meshes/wheel_right_link.STL"/>
             </geometry>
         </visual>
@@ -79,5 +79,5 @@
             <geometry>
                 <!-- <mesh filename="package://robot_description/meshes/wheel_left_link.STL" scale="1 1 1"/> -->
-                <mesh filename="$(find robot_description)/meshes/wheel_left_link.STL"/>
+                <mesh filename="file://$(find robot_description)/meshes/wheel_left_link.STL"/>
             </geometry>
         </visual>
@@ -108,5 +108,5 @@
            <geometry>
                <!-- <mesh filename="package://robot_description/meshes/caster_front_link.STL" scale="1 1 1"/> -->
-                <mesh filename="$(find robot_description)/meshes/caster_front_link.STL"/>
+                <mesh filename="file://$(find robot_description)/meshes/caster_front_link.STL"/>
             </geometry>
         </visual>
@@ -141,5 +141,5 @@
             <geometry>
                 <!-- <mesh filename="package://robot_description/meshes/caster_rear_link.STL" scale="1 1 1"/> -->
-                <mesh filename="$(find robot_description)/meshes/caster_rear_link.STL"/>
+                <mesh filename="file://$(find robot_description)/meshes/caster_rear_link.STL"/>
             </geometry>
         </visual>

File: src/robot_description/urdf/camera.xacro (robot description, xacro)
@@ -28,3 +28,15 @@
         <origin xyz="0.07 0 0.03" rpy="0 0 0" />
     </joint>
+    <!-- gazebo plugin for camera -->
+     <gazebo reference = "camera_link">
+        <material>Gazebo/Grey</material>
+        <sensor name = "camera_sensor" type="camera">
+            <pose>0 0 0 0 0 0 </pose>
+            <visualize>true</visualize>
+            <update_rate>10.0</update_rate>
+            <plugin name="camera_controller" filename="libgazebo_ros_camera.so">
+                <frame_name>camera_link</frame_name>
+            </plugin>
+        </sensor>
+     </gazebo>
 </robot>

Commit message: new models for the world added , ros2_control configured

File: src/robot_description/urdf/bumperbot.urdf.xacro (robot description, xacro)
@@ -1,4 +1,4 @@
 <?xml version="1.0"?>
-<robot xmlns:xacro="http://www.ros.org/wiki/xacro" name="bumberbot">
+<robot xmlns:xacro="http://www.ros.org/wiki/xacro" name="bumperbot">
     <xacro:arg name="is_ignition" default="true"/>
     <!-- Include gazebo parameters -->
@@ -7,5 +7,5 @@
     <xacro:include filename="$(find robot_description)/urdf/camera.xacro"/>
     <!-- ROS2 control -->
-    <!-- <xacro:include filename="$(find robot_description)/urdf/bumperbot_ros2_control.xacro"/> -->
+    <xacro:include filename="$(find robot_description)/urdf/bumperbot_ros2_control.xacro"/>
     <link name="base_footprint"/>
     <link name="base_link">
@@ -132,9 +132,4 @@
                     izz="1.00967486676306e-10"/>
         </inertial>
-        <inertial>
-            <origin xyz="0.0 0.0 0.0" rpy="0.0 0.0 0.0"/>
-            <mass value="0.0"/>
-            <inertia ixx="0.0" ixy="0.0" ixz="0.0" iyy="0.0" iyz="0.0" izz="0.0"/>
-        </inertial>
         <visual>
             <origin xyz="0.0 0.0 0.0" rpy="0.0 0.0 0.0"/>

File: src/robot_description/urdf/bumperbot_gazebo.xacro (robot description, xacro)
@@ -69,15 +69,9 @@
         <maxvel>0.1</maxvel>
     </gazebo>
-    <!-- <gazebo>
-        <xacro:if value="$(arg is_ignition)">
-            <plugin filename="ign_ros2_control-system" name="ign_ros2_control::IgnitionROS2ControlPlugin">
-                <parameters>$(find bumperbot_controller)/config/bumperbot_controllers.yaml</parameters>
-            </plugin>
-        </xacro:if>
-        <xacro:unless value="$(arg is_ignition)">
-            <plugin filename="gz_ros2_control-system" name="gz_ros2_control::GazeboSimROS2ControlPlugin">
-                <parameters>$(find bumperbot_controller)/config/bumperbot_controllers.yaml</parameters>
-            </plugin>
-        </xacro:unless>
-    </gazebo> -->
+    <gazebo>
+        <plugin filename="libgazebo_ros2_control.so" name="gazebo_ros2_control">
+            <parameters>$(find bumperbot_controller)/config/bumperbot_controllers.yaml</parameters>
+            <!-- <robot_param>robot_description</robot_param> -->
+        </plugin>
+    </gazebo>
 </robot>

File: src/robot_description/urdf/bumperbot_ros2_control.xacro (robot description, xacro)
@@ -1,16 +1,11 @@
 <?xml version="1.0"?>
 <robot xmlns:xacro="http://www.ros.org/wiki/xacro" name="bumperbot">
+    <!-- ROS2 Control Setup -->
     <ros2_control name="RobotSystem" type="system">
-        <xacro:if value="$(arg is_ignition)">
-            <hardware>
-                <plugin>ign_ros2_control/IgnitionSystem</plugin>
-            </hardware>
-        </xacro:if>
-        <xacro:unless value="$(arg is_ignition)">
-            <hardware>
-                <plugin>gz_ros2_control/GazeboSimSystem</plugin>
-            </hardware>
-        </xacro:unless>
-        <joint name="wheel_left_joint">
+        <hardware>
+            <plugin>gazebo_ros2_control/GazeboSystem</plugin>
+        </hardware>
+        <!-- Right wheel joint -->
+        <joint name="wheel_right_joint">
             <command_interface name="velocity">
                 <param name="min">-1</param>
@@ -20,5 +15,6 @@
             <state_interface name="velocity"/>
         </joint>
-        <joint name="wheel_right_joint">
+        <!-- Left wheel joint -->
+        <joint name="wheel_left_joint">
             <command_interface name="velocity">
                 <param name="min">-1</param>

File: src/robot_description/urdf/camera.xacro (robot description, xacro)
@@ -26,5 +26,5 @@
         <parent link="base_link" />
         <child link="camera_link" />
-        <origin xyz="0.07 0 0.03" rpy="0 0 0" />
+        <origin xyz="0.07 0 0.07" rpy="0 0 0" />
     </joint>
     <!-- gazebo plugin for camera -->
@@ -33,5 +33,5 @@
         <sensor name = "camera_sensor" type="camera">
             <pose>0 0 0 0 0 0 </pose>
-            <visualize>true</visualize>
+            <visualize>false</visualize>
             <update_rate>10.0</update_rate>
             <plugin name="camera_controller" filename="libgazebo_ros_camera.so">

Commit message: aruco markers added to the simulation

File: src/robot_description/urdf/bumperbot.urdf.xacro (robot description, xacro)
@@ -1,4 +1,4 @@
 <?xml version="1.0"?>
-<robot xmlns:xacro="http://www.ros.org/wiki/xacro" name="bumperbot">
+<robot xmlns:xacro="http://www.ros.org/wiki/xacro" name="my_robot">
     <xacro:arg name="is_ignition" default="true"/>
     <!-- Include gazebo parameters -->

File: src/robot_description/urdf/bumperbot_gazebo.xacro (robot description, xacro)
@@ -1,4 +1,4 @@
 <?xml version="1.0"?>
-<robot xmlns:xacro="http://www.ros.org/wiki/xacro" name="bumperbot">
+<robot xmlns:xacro="http://www.ros.org/wiki/xacro" name="my_robot">
     <!-- <gazebo reference="wheel_right_link">
         <mu1>100000000000000.0</mu1>
@@ -35,4 +35,7 @@
         <maxvel>0.1</maxvel>
     </gazebo> -->
+    <gazebo reference="base_link">
+        <material>Gazebo/Black</material>
+    </gazebo>
      <gazebo reference="wheel_right_link">
         <mu1>1.0</mu1>
@@ -71,5 +74,5 @@
     <gazebo>
         <plugin filename="libgazebo_ros2_control.so" name="gazebo_ros2_control">
-            <parameters>$(find bumperbot_controller)/config/bumperbot_controllers.yaml</parameters>
+            <parameters>$(find bumperbot_controller)/config/bumperbot_controller.yaml</parameters>
             <!-- <robot_param>robot_description</robot_param> -->
         </plugin>

File: src/robot_description/urdf/bumperbot_ros2_control.xacro (robot description, xacro)
@@ -1,4 +1,4 @@
 <?xml version="1.0"?>
-<robot xmlns:xacro="http://www.ros.org/wiki/xacro" name="bumperbot">
+<robot xmlns:xacro="http://www.ros.org/wiki/xacro" name="my_robot">
     <!-- ROS2 Control Setup -->
     <ros2_control name="GazeboSystem" type="system">

File: src/robot_description/urdf/camera.xacro (robot description, xacro)
@@ -30,11 +30,42 @@
     <!-- gazebo plugin for camera -->
      <gazebo reference = "camera_link">
-        <material>Gazebo/Grey</material>
+        <material>Gazebo/Blue</material>
         <sensor name = "camera_sensor" type="camera">
             <pose>0 0 0 0 0 0 </pose>
             <visualize>false</visualize>
             <update_rate>10.0</update_rate>
+            <camera name="head">
+                <horizontal_fov>1.3962634</horizontal_fov>
+                <image>
+                <width>1280</width>
+                <height>720</height>
+                <format>R8G8B8</format>
+                </image>
+                <clip>
+                <near>0.01</near>
+                <far>5</far>
+                </clip>
+                <noise>
+                <type>gaussian</type>
+                <!-- Noise is sampled independently per pixel on each frame.
+                    That pixel's noise value is added to each of its color
+                    channels, which at that point lie in the range [0,1]. -->
+                <mean>0.0</mean>
+                <stddev>0.007</stddev>
+                </noise>
+            </camera>
             <plugin name="camera_controller" filename="libgazebo_ros_camera.so">
-                <frame_name>camera_link</frame_name>
+                <alwaysOn>true</alwaysOn>
+                <updateRate>0.0</updateRate>
+                <cameraName>my_robot/camera1</cameraName>
+                <imageTopicName>image_raw</imageTopicName>
+                <cameraInfoTopicName>camera_info</cameraInfoTopicName>
+                <frameName>camera_link</frameName>
+                <hackBaseline>0.07</hackBaseline>
+                <distortionK1>0.0</distortionK1>
+                <distortionK2>0.0</distortionK2>
+                <distortionK3>0.0</distortionK3>
+                <distortionT1>0.0</distortionT1>
+                <distortionT2>0.0</distortionT2>
             </plugin>
         </sensor>
